File: modkey/modkey.kicad_pcb (KiCad board)
At the start: 2 copper layers, 19.1 x 19 mm, 12 parts, among them J1 Conn_01x04, J2 Conn_01x04, J3 Conn_01x04, J4 Conn_01x04, SW1 SW_Push, U1 ATtiny85-20SU

Commit message: pull up with less than the force of a thousand suns
Parts:
- R1, R2: value 4k7 -> Open
Changed lines of the file:
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@@
       (effects (font (size 1 1) (thickness 0.15)) (justify mirror))
     )
-    (fp_text value 4k7 (at 0 -1.65) (layer B.Fab)
+    (fp_text value Open (at 0 -1.65) (layer B.Fab)
       (effects (font (size 1 1) (thickness 0.15)) (justify mirror))
     )
@@
       (effects (font (size 1 1) (thickness 0.15)) (justify mirror))
     )
-    (fp_text value 4k7 (at 0 -1.65) (layer B.Fab)
+    (fp_text value Open (at 0 -1.65) (layer B.Fab)
       (effects (font (size 1 1) (thickness 0.15)) (justify mirror))
     )
