File: modkey/modkey.kicad_pcb (KiCad board)
At the start: 2 copper layers, 19.1 x 19 mm, 12 parts, among them J1 Conn_01x04, J2 Conn_01x04, J3 Conn_01x04, J4 Conn_01x04, SW1 SW_Push, U1 ATtiny85-20SU

Commit message: update
Parts:
- R1: value Open -> 1k; footprint Resistor_SMD:R_0805_2012Metric_Pad1.15x1.40mm_HandSolder -> Resistor_SMD:R_0805_2012Metric_Pad1.20x1.40mm_HandSolder
- R2: value Open -> 10k; footprint Resistor_SMD:R_0805_2012Metric_Pad1.15x1.40mm_HandSolder -> Resistor_SMD:R_0805_2012Metric_Pad1.20x1.40mm_HandSolder
- moved R3 13.0 mm to (136.0, 92.0), turned to 270 degrees
- moved R1 12.7 mm to (146.5, 87.0), turned to 0 degrees
- moved R2 10.3 mm to (135.5, 80.0)
- moved R5 1.68 mm to (148.0, 90.0), turned to 270 degrees
- moved R4 1.06 mm to (150.0, 91.0), turned to 270 degrees
Connections:
- net /B renamed Net-(D1-Pad2)
- net /G renamed Net-(D1-Pad3)
- net /R renamed Net-(D1-Pad4)
- R1 pad 1: SDA -> KEY
- R2 pad 1: SCL -> Net-(R2-Pad1)
- R2 pad 2: +5V -> GND
- R3 pad 2: /PB4 -> R
- R4 pad 2: /PB3 -> G
- R5 pad 2: /PB5 -> B
- SW1 pad 1: /PB1 -> KEY
- SW1 pad 2: GND -> Net-(R2-Pad1)
- U1 pad 1: /PB5 -> KEY
- U1 pad 2: /PB3 -> B
- U1 pad 3: /PB4 -> G
- U1 pad 6: /PB1 -> R
Routing:
- net /PB1: track 27.7 -> 0.00 mm, vias 2 -> 0
- net KEY: track 0.00 -> 20.3 mm
- net Net-(R2-Pad1): track 0.00 -> 7.21 mm, vias 0 -> 1
- net +5V: track 43.4 -> 36.9 mm, vias 6 -> 7
- net G: track 0.00 -> 4.61 mm
- net GND: track 41.0 -> 45.2 mm, vias 6 -> 8
- net Net-(D1-Pad4): track 9.86 -> 5.92 mm
- net R: track 0.00 -> 2.86 mm
- net /PB4: track 2.83 -> 0.00 mm
- net SCL: track 42.5 -> 39.7 mm, vias 6 -> 7
- net B: track 0.00 -> 2.72 mm
- net /PB5: track 2.56 -> 0.00 mm
- net /PB3: track 2.54 -> 0.00 mm
- net SDA: track 41.4 -> 39.2 mm, vias 6 -> 5
- net Net-(D1-Pad2): track 7.66 -> 6.90 mm
Other:
- net class Default: trace_width 0.25 -> 0.1524

Commit message: cleanup
Parts:
- added ?: , Aesthetics:OSHW-LOGO-M, F.Cu at (147.5, 91.0)
- D1: value LED_ABGR -> ABGR
Other:
- board text added: "5V SDA SCL"
- board text added: "GND"
- board text added: "SCL SDA 5V"
