File: modctrl/modctrl.kicad_pcb (KiCad board)
At the start: 2 copper layers, 19 x 19 mm, 19 parts, among them J1 USB_C_Receptacle, J2 Conn_01x04, SW1 SW_Push, U1 ATmega32U4-AU, Y1 16MHz

Commit message: pull up with less than the force of a thousand suns
Parts:
- added R7: 4k7, Resistor_SMD:R_0805_2012Metric_Pad1.15x1.40mm_HandSolder, F.Cu at (137.3, 65.9)
- added R8: 4k7, Resistor_SMD:R_0805_2012Metric_Pad1.15x1.40mm_HandSolder, F.Cu at (139.3, 65.9)
Routing:
- net +5V: track 82.2 -> 71.2 mm, vias 6 -> 7
- net SDA: track 2.02 -> 12.2 mm
- net SCL: track 2.71 -> 10.7 mm
- net GND: track 119.0 -> 116.1 mm, vias 7 -> 6

Commit message: cleanup
Parts:
- added ?: , Aesthetics:OSHW-LOGO-MINI, F.Cu at (139.5, 51.5)
- C2, C3: value 22pF -> 22p
- C4, C5: value 100nF -> 100n
- C6: value 10μF -> 10μ
- C7: value 1μF -> 1μ
- R1, R2: value 5.1kΩ -> 5.1k
- R3: value 22Ω -> 22
- R5, R6: value 10kΩ -> 10k
