File: modjoy/modjoy.kicad_pcb (KiCad board)
At the start: 2 copper layers, 19.1 x 19 mm, 10 parts, among them J1 Conn_01x04, J2 Conn_01x04, J3 Conn_01x04, U1 ATtiny85-20SU

Commit message: update
Routing:
- net /PB1: track 0.00 -> 8.02 mm

Commit message: cleanup
Parts:
- added ?: , Aesthetics:OSHW-LOGO-L, F.Cu at (152.0, 92.5)
