File: modjoy/modjoy.sch (KiCad schematic (older format))
At the start: 10 parts, among them J1 Conn_01x04, J2 Conn_01x04, J3 Conn_01x04, U1 ATtiny85-20SU

Commit message: cleanup
Changed lines of the file:
@@
 U 1 1 5E44387B
 P 4100 4300
-F 0 "R1" V 3900 4450 50  0000 C CNN
-F 1 "220" V 4000 4450 50  0000 C CNN
+F 0 "R1" V 4000 4400 50  0000 C CNN
+F 1 "220" V 4100 4300 50  0000 C CNN
 F 2 "Resistor_SMD:R_0805_2012Metric_Pad1.15x1.40mm_HandSolder" V 4030 4300 50  0001 C CNN
 F 3 "~" H 4100 4300 50  0001 C CNN
